File: KiCAD/current-modules/8stepsequencer/8stepsequencer.kicad_sch (KiCad schematic)
At the start: 57 parts, among them SW10 s4_mute, SW11 s3_mute, SW12 s2_mute, SW13 s1_mute, SW14 SW_DPST, SW2 SW_Rotary_1x12, SW3 tuning_button, SW4 tuning_mode, SW6 s8_mute, SW7 s7_mute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

Commit message: Sequencer Tweaks
Additions:
- Text IO labels
Changes:
- Replaced 2 related SPSTs with a DPST
Removals:
- None
NOTES:
- Still needs audio jack IO peripherals
Parts:
- removed SW14: SW_DPST, symbol Switch:SW_DPST
- added SW5: Seq_pwr, symbol Switch:SW_SPST
Connections:
- net at C4.1, SW3.1, U3.16 (VDD)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: now also SW5.2 (B)
- net at C5.1, U6.3 (OUT): now also SW5.1 (A)
Other:
- note removed: "clock in*"
- note removed: "gate out"
- note removed: "output"
Changed lines of the file:
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@@
 	(generator_version "10.0")
 	(paper "A4")
-	(text "clock in*"
-		(exclude_from_sim no)
-		(at 61.722 51.816 0)
-		(effects
-			(font
-				(size 1.27 1.27)
-			)
-		)
-	)
-	(text "gate out"
-		(exclude_from_sim no)
-		(at 79.248 72.898 0)
-		(effects
-			(font
-				(size 1.27 1.27)
-			)
-		)
-	)
-	(text "clock in*"
-		(exclude_from_sim no)
-		(at 22.352 86.614 0)
-		(effects
-			(font
-				(size 1.27 1.27)
-			)
-		)
-	)
-	(text "output"
-		(exclude_from_sim no)
-		(at 70.612 17.272 0)
-		(effects
-			(font
-				(size 1.27 1.27)
-			)
-		)
-	)
 	(junction
 		(at 212.09 71.12)
@@
 	)
 	(junction
-		(at 71.12 85.09)
-		(diameter 0)
-		(color 0 0 0 0)
-	)
-	(junction
 		(at 69.85 72.39)
 		(diameter 0)
@@
 	)
 	(junction
+		(at 73.66 30.48)
+		(diameter 0)
+		(color 0 0 0 0)
+	)
+	(junction
 		(at 218.44 109.22)
 		(diameter 0)
@@
 	)
 	(junction
-		(at 92.71 30.48)
-		(diameter 0)
-		(color 0 0 0 0)
-	)
-	(junction
 		(at 40.64 40.64)
 		(diameter 0)
@@
 	(wire
 		(pts
-			(xy 63.5 30.48) (xy 63.5 26.67)
-		)
-		(stroke
-			(width 0)
-			(type default)
-		)
-	)
-	(wire
-		(pts
 			(xy 180.34 144.78) (xy 180.34 139.7)
 		)
@@
 	(wire
 		(pts
-			(xy 264.16 19.05) (xy 92.71 19.05)
-		)
-		(stroke
-			(width 0)
-			(type default)
-		)
-	)
-	(wire
-		(pts
 			(xy 134.62 78.74) (xy 134.62 81.28)
 		)
@@
 	(wire
 		(pts
-			(xy 71.12 85.09) (xy 74.93 85.09)
-		)
-		(stroke
-			(width 0)
-			(type default)
-		)
-	)
-	(wire
-		(pts
 			(xy 147.32 67.31) (xy 212.09 67.31)
 		)
@@
 	(wire
 		(pts
-			(xy 71.12 74.93) (xy 78.74 74.93)
-		)
-		(stroke
-			(width 0)
-			(type default)
-		)
-	)
-	(wire
-		(pts
 			(xy 218.44 101.6) (xy 218.44 109.22)
 		)
@@
 	(wire
 		(pts
-			(xy 64.77 85.09) (xy 71.12 85.09)
-		)
-		(stroke
-			(width 0)
-			(type default)
-		)
-	)
-	(wire
-		(pts
-			(xy 69.85 19.05) (xy 69.85 21.59)
+			(xy 64.77 85.09) (xy 74.93 85.09)
 		)
 		(stroke
@@
 	(wire
 		(pts
-			(xy 92.71 30.48) (xy 133.35 30.48)
-		)
-		(stroke
-			(width 0)
-			(type default)
-		)
-	)
-	(wire
-		(pts
 			(xy 19.05 77.47) (xy 19.05 60.96)
 		)
@@
 	(wire
 		(pts
-			(xy 92.71 26.67) (xy 92.71 30.48)
-		)
-		(stroke
-			(width 0)
-			(type default)
-		)
-	)
-	(wire
-		(pts
 			(xy 184.15 86.36) (xy 184.15 58.42)
 		)
@@
 	(wire
 		(pts
-			(xy 71.12 85.09) (xy 71.12 74.93)
-		)
-		(stroke
-			(width 0)
-			(type default)
-		)
-	)
-	(wire
-		(pts
 			(xy 68.58 40.64) (xy 60.96 40.64)
 		)
@@
 	(wire
 		(pts
-			(xy 63.5 26.67) (xy 82.55 26.67)
-		)
-		(stroke
-			(width 0)
-			(type default)
-		)
-	)
-	(wire
-		(pts
 			(xy 135.89 96.52) (xy 154.94 96.52)
 		)
@@
 	(wire
 		(pts
-			(xy 73.66 30.48) (xy 92.71 30.48)
+			(xy 73.66 30.48) (xy 133.35 30.48)
 		)
 		(stroke
@@
 	(wire
 		(pts
-			(xy 82.55 21.59) (xy 69.85 21.59)
-		)
-		(stroke
-			(width 0)
-			(type default)
-		)
-	)
-	(wire
-		(pts
 			(xy 201.93 114.3) (xy 196.85 114.3)
 		)
@@
 	(wire
 		(pts
-			(xy 264.16 73.66) (xy 264.16 19.05)
-		)
-		(stroke
-			(width 0)
-			(type default)
-		)
-	)
-	(wire
-		(pts
 			(xy 85.09 87.63) (xy 85.09 92.71)
 		)
@@
 	(wire
 		(pts
-			(xy 92.71 19.05) (xy 92.71 21.59)
-		)
-		(stroke
-			(width 0)
-			(type default)
-		)
-	)
-	(wire
-		(pts
 			(xy 199.39 124.46) (xy 205.74 124.46)
 		)
@@
 	)
 	(symbol
-		(lib_id "Switch:SW_DPST")
-		(at 87.63 24.13 0)
-		(unit 1)
-		(body_style 1)
-		(exclude_from_sim no)
-		(in_bom yes)
-		(on_board yes)
-		(in_pos_files yes)
-		(dnp no)
-		(fields_autoplaced yes)
-		(property "Reference" "SW14"
-			(at 87.63 15.24 0)
-			(show_name no)
-			(do_not_autoplace no)
-			(effects
-				(font
-					(size 1.27 1.27)
-				)
-			)
-		)
-		(property "Value" "SW_DPST"
-			(at 87.63 17.78 0)
-			(show_name no)
-			(do_not_autoplace no)
-			(effects
-				(font
-					(size 1.27 1.27)
-				)
-			)
-		)
-		(property "Footprint" ""
-			(at 87.63 24.13 0)
-			(hide yes)
-			(show_name no)
-			(do_not_autoplace no)
-			(effects
-				(font
-					(size 1.27 1.27)
-				)
-			)
-		)
-		(property "Datasheet" ""
-			(at 87.63 24.13 0)
-			(hide yes)
-			(show_name no)
-			(do_not_autoplace no)
-			(effects
-				(font
-					(size 1.27 1.27)
-				)
-			)
-		)
-		(property "Description" "Double Pole Single Throw (DPST) Switch"
-			(at 87.63 24.13 0)
-			(hide yes)
-			(show_name no)
-			(do_not_autoplace no)
-			(effects
-				(font
-					(size 1.27 1.27)
-				)
-			)
-		)
-		(pin "4"
-		)
-		(pin "3"
-		)
-		(pin "2"
-		)
-		(pin "1"
-		)
-		(instances
-			(project "synth-allmodules"
-				(path "/f3152922-b7ee-45aa-a88a-669787bc63c5/fa0c7a75-82fb-4569-92a3-ed5c40158d6b"
-					(reference "SW14")
-					(unit 1)
-				)
-			)
-		)
-	)
-	(symbol
 		(lib_id "Device:C_Polarized")
 		(at 19.05 57.15 180)
@@
 					(unit 1)
 				)
+			)
+		)
+	)
+	(symbol
+		(lib_id "Switch:SW_SPST")
+		(at 68.58 30.48 0)
+		(unit 1)
+		(body_style 1)
+		(exclude_from_sim no)
+		(in_bom yes)
+		(on_board yes)
+		(in_pos_files yes)
+		(dnp no)
+		(fields_autoplaced yes)
+		(property "Reference" "SW5"
+			(at 68.58 24.13 0)
+			(show_name no)
+			(do_not_autoplace no)
+			(effects
+				(font
+					(size 1.27 1.27)
+				)
+			)
+		)
+		(property "Value" "Seq_pwr"
+			(at 68.58 26.67 0)
+			(show_name no)
+			(do_not_autoplace no)
+			(effects
+				(font
+					(size 1.27 1.27)
+				)
+			)
+		)
+		(property "Footprint" ""
+			(at 68.58 30.48 0)
+			(hide yes)
+			(show_name no)
+			(do_not_autoplace no)
+			(effects
+				(font
+					(size 1.27 1.27)
+				)
+			)
+		)
+		(property "Datasheet" ""
+			(at 68.58 30.48 0)
+			(hide yes)
+			(show_name no)
+			(do_not_autoplace no)
+			(effects
+				(font
+					(size 1.27 1.27)
+				)
+			)
+		)
+		(property "Description" "Single Pole Single Throw (SPST) switch"
+			(at 68.58 30.48 0)
+			(hide yes)
+			(show_name no)
+			(do_not_autoplace no)
+			(effects
+				(font
+					(size 1.27 1.27)
+				)
+			)
+		)
+		(pin "2"
+		)
+		(pin "1"
+		)
+		(instances
+			(project "synth-allmodules"
+				(path "/f3152922-b7ee-45aa-a88a-669787bc63c5/fa0c7a75-82fb-4569-92a3-ed5c40158d6b"
+					(reference "SW5")
+					(unit 1)
+				)
