File: KiCAD/current-modules/synth-allmodules/bass.kicad_sch (KiCad schematic)
At the start: 0 parts

Commit message: Added bass module
Additions:
- Bass module minus audio jacks
Changes:
- None
Removals:
- None
Parts:
- added C10, C12, C14, C18, C19: 2.2u, symbol Device:C_Polarized
- added C11: 4.7n, symbol Device:C
- added C13, C15, C22, C23, C24, C25: 10n, symbol Device:C
- added C16, C17: 100n, symbol Device:C
- added C20, C21: 10u, symbol Device:C_Polarized
- added C9: 1n, symbol Device:C
- added D24, D26, D27, D28, D29: 1N4148, Diode_THT:D_DO-35_SOD27_P7.62mm_Horizontal, symbol Diode:1N4148
- added D25: LED, symbol Device:LED
- added Q5, Q8: 2N3904, Package_TO_SOT_THT:TO-92_Inline, symbol Transistor_BJT:2N3904
- added Q6, Q7: 2N3906, Package_TO_SOT_THT:TO-92_Inline, symbol Transistor_BJT:2N3906
- added R28: 100R, symbol Device:R
- added R29, R39, R43: 20K, symbol Device:R
- added R30: 1M, symbol Device:R
- added R31: 1K, symbol Device:R
- added R32, R45, R48: 10K, symbol Device:R
- added R33, R40, R49, R50, R51: 100K, symbol Device:R
- added R34, R44: 56K, symbol Device:R
- added R35: 27K, symbol Device:R
- added R36: 3.3K, symbol Device:R
- added R37: 2K, symbol Device:R
- added R38: 5.1K, symbol Device:R
- added R41, R42: 220R, symbol Device:R
- added R46: 220K, symbol Device:R
- added R47: 1.5K, symbol Device:R
- added RV15, RV17, RV21, RV23: 10K, symbol Device:R_Potentiometer
- added RV16: 500K, symbol Device:R_Potentiometer
- added RV18, RV19, RV20, RV22: 100K, symbol Device:R_Potentiometer
- added U7: TL072, symbol Amplifier_Operational:TL072
- added U8: LM13700, symbol Amplifier_Operational:LM13700
Connections:
- new net: C11.1, D26.2 (A), D27.1 (K), U8.3 (+)
- new net: Q5.1 (E), R43.1, RV17.1
- new net: Q5.2 (B), R32.2
- new net: C13.2, R44.2, U8.10, U8.12
- new net: Q7.1 (E), R43.2
- new net: C17.1, R48.1, RV21.3
- new net: R33.1, RV17.2
- new net: Q6.1 (E), R33.2, R34.2, R35.1
- new net: R29.1, RV15.1
- new net: RV15.2, U7.2 (-)
- new net: R28.2, RV15.3
- new net: R49.2, R50.1, R51.1, U7.6 (-)
- new net: R50.2, RV22.2
- new net: R34.1, RV18.2
- new net: C19.1, R51.2, U7.7
- new net: C10.1, D24.1 (K), R31.2, R32.1
- new net: Q8.2 (B), R46.1
- new net: Q8.3 (C), R47.1
- new net: C14.2, R45.2, U8.9
- new net: D25.1 (K), R47.2
- new net: C9.2, R30.2, U7.3 (+)
- new net: C14.1, RV20.1
- new net: R49.1, RV20.2
- new net: Q7.3 (C), U8.16
- new net: R35.2, RV19.2
- new net: C18.2, RV22.1
- new net: C16.2, RV21.1
- new net: C18.1, RV21.2
- new net: C12.1, R40.1
- new net: R40.2, R41.2, U8.14 (+)
- new net: C16.1, D29.1 (K), R48.2
- new net: R36.2, RV19.1
- new net: R31.1, RV16.3
- new net: R37.2, R39.1, U8.4 (-)
- new net: R42.2, U8.13 (-)
- new net: Q6.3 (C), U8.1
- new net: D24.2 (A), D28.2 (A), D29.2 (A), U7.1
- new net: C15.1, D28.1 (K), R46.2
- new net: C11.2, U8.5, U8.7
- new net: C12.2, R38.2, R39.2, U8.8
- new net: C19.2, RV23.1
- new net GND: C10.2, C13.1, C15.2, C17.2, C20.2, C21.1, C22.1, C23.1, C24.2, C25.2, D26.1 (K), D27.2 (A), Q6.2 (B), Q7.2 (B), Q8.1 (E), R28.1, R30.1, R36.1, R37.1, R41.1, R42.1, R44.1, RV16.1, RV16.2, RV17.3, RV18.3, RV20.3, RV22.3, RV23.3, U7.5 (+)
- new net VCC: C20.1, C22.2, C23.2, D25.2 (A), Q5.3 (C), R29.2, RV19.3, U7.8 (V+), U8.11 (V+)
- new net VSS: C21.2, C24.1, C25.1, R38.1, R45.1, U7.4 (V-), U8.6 (V-)
Other:
- note added: "Decay"
- note added: "Impact tone"
- note added: "Impact vol"
- note added: "Master vol"
- note added: "Pitch"
- note added: "Range"
- note added: "Shell vol"
- note added: "Sweep"
- note added: "Trigger"
