File: KiCAD/current-modules/synth-allmodules/bass.kicad_sch (KiCad schematic)
At the start: 62 parts, among them Q5 2N3904, Q6 2N3906, Q7 2N3906, Q8 2N3904, U7 TL072, U8 LM13700

Commit message: Audio Jacks
Additions:
- Audio jack IOs for all sheets
Changes:
- None
Removals:
- None
Parts:
- added J10: TRIGGER, Connector_PinHeader_2.54mm:PinHeader_1x02_P2.54mm_Vertical, symbol Connector_Generic:Conn_01x02
- added J11: CV, Connector_PinHeader_2.54mm:PinHeader_1x02_P2.54mm_Vertical, symbol Connector_Generic:Conn_01x02
- added J12: OUTPUT, Connector_PinHeader_2.54mm:PinHeader_1x02_P2.54mm_Vertical, symbol Connector_Generic:Conn_01x02
Connections:
- net GND: now also J10.2 (Pin_2), J11.2 (Pin_2), J12.2 (Pin_2)
- net at RV18.1: now also J11.1 (Pin_1)
- net at C9.1: now also J10.1 (Pin_1)
- net at RV23.2: now also J12.1 (Pin_1)
Other:
- note added: "Output"
