File: KiCAD/current-modules/synth-allmodules/8stepsequencer.kicad_sch (KiCad schematic)
At the start: 57 parts, among them SW10 s4_mute, SW11 s3_mute, SW12 s2_mute, SW13 s1_mute, SW14 SW_DPST, SW2 SW_Rotary_1x12, SW3 tuning_button, SW4 tuning_mode, SW6 s8_mute, SW7 s7_mute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

Commit message: Label changes
Other:
- note added: "OUT"
- note removed: "output"
Changed lines of the file:
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@@
 		)
 	)
-	(text "output"
+	(text "OUT"
 		(exclude_from_sim no)
 		(at 70.612 17.272 0)
