File: KiCAD/current-modules/synth-allmodules/8stepsequencer.kicad_sch (KiCad schematic)
At the start: 57 parts, among them SW10 s4_mute, SW11 s3_mute, SW12 s2_mute, SW13 s1_mute, SW14 SW_DPST, SW2 SW_Rotary_1x12, SW3 tuning_button, SW4 tuning_mode, SW6 s8_mute, SW7 s7_mute, SW8 s6_mute, SW9 s5_mute, U3 CD4017BEE4, U4 CD40106BEE4, U5 TL072, U6 L7808

Commit message: Audio Jacks
Additions:
- Audio jack IOs for all sheets
Changes:
- None
Removals:
- None
Parts:
- added J7: CLOCK_IN, Connector_PinHeader_2.54mm:PinHeader_1x03_P2.54mm_Vertical, symbol Connector_Generic:Conn_01x03
- added J8: GATE_OUT, Connector_PinHeader_2.54mm:PinHeader_1x02_P2.54mm_Vertical, symbol Connector_Generic:Conn_01x02
- added J9: CV_OUT, Connector_PinHeader_2.54mm:PinHeader_1x02_P2.54mm_Vertical, symbol Connector_Generic:Conn_01x02
Connections:
- net GND: now also J7.3 (Pin_3), J8.2 (Pin_2), J9.2 (Pin_2)
- net at SW4.3 (C), U4.8 (J=~D): now also J8.1 (Pin_1)
- net at SW14.3: now also J9.1 (Pin_1)
- net at U4.11 (E): now also J7.1 (Pin_1)
- net CLK_NORMAL: now reaches RV6.3, U4.2 (G=~A)
- net CLK_NORMAL: now also J7.2 (Pin_2)
