File: KiCAD/current-modules/synth-allmodules/808kick.kicad_sch (KiCad schematic)
At the start: 0 parts

Commit message: First Draft of 808
Additions:
- Draft of 808 Kick module
Changes:
- None
Removals:
- None
Parts:
- added C1, C10, C2, C9: 100n, symbol Device:C
- added C3: 33n, symbol Device:C
- added C4, C5: 15n, symbol Device:C
- added C6: 33u, symbol Device:C_Polarized
- added C7: 470n, symbol Device:C
- added D1, D2, D3: 1N4148, symbol Diode:1N4148
- added D4: LED, symbol Device:LED
- added Q1: 2N3906, symbol Transistor_BJT:2N3906
- added Q2: 2N3904, symbol Transistor_BJT:2N3904
- added R1, R7: 22K, symbol Device:R
- added R10: 6.8K, symbol Device:R
- added R11: 470K, symbol Device:R
- added R12, R4, R8: 1M, symbol Device:R
- added R13: 330K, symbol Device:R
- added R14, R15, R3: 47K, symbol Device:R
- added R16, R19: 680R, symbol Device:R
- added R17: 20K, symbol Device:R
- added R18, R2: 10K, symbol Device:R
- added R20: 1K, symbol Device:R
- added R5: 2.7K, symbol Device:R
- added R6: 8.2K, symbol Device:R
- added R9: 100K, symbol Device:R
- added RV1: 10K, symbol Device:R_Potentiometer
- added RVdecay: 500K (panel: Decay), symbol Device:R_Potentiometer
- added RVlevel: 10K (panel: Level), symbol Device:R_Potentiometer
- added RVpitch: 100K (panel: Pitch), symbol Device:R_Potentiometer
- added RVtone: 5K (panel: Tone), symbol Device:R_Potentiometer
- added U1: TL074, symbol Amplifier_Operational:TL074
Connections:
- new net: D4.2 (A), R20.1
- new net: R12.1, R13.2, U1.1
- new net: C5.1, R12.2, U1.3 (+)
- new net: Q2.2 (B), RV1.1, U1.13 (-)
- new net: Q1.1 (E), RV1.2, RV1.3
- new net: R15.1, RVdecay.2, RVdecay.3
- new net: C6.2, R11.1, R14.1, R15.2, U1.5 (+)
- new net: C3.2, R7.1
- new net: Q2.1 (E), R4.1, R5.2
- new net: R13.1, R14.2
- new net: C4.1, C5.2, RVtone.2, RVtone.3
- new net: C4.2, R10.1, R11.2
- new net: R20.2, U1.12 (+), U1.14
- new net: C1.2, D1.1 (K), D1.2 (A)
- new net: Q1.2 (B), R1.1, R2.2, R3.1
- new net: R17.2, R18.1, U1.10 (+)
- new net: D3.2 (A), R16.1, R18.2
- new net: C7.1, R16.2, RVlevel.2, RVlevel.3
- new net: C6.1, C7.2, RVdecay.1, U1.7
- new net: R10.2, R6.1, R8.1, R9.2
- new net: C2.1, C2.2, R5.1, R6.2
- new net: C1.1, R1.2
- new net: R9.1, RVpitch.2, RVpitch.3
- new net: C3.1, D2.2 (A), R8.2
- new net: R17.1, R19.2, U1.8
- new net GND: C10.1, C9.1, D2.1 (K), D3.1 (K), D4.1 (K), Q2.3 (C), R2.1, RVlevel.1, RVpitch.1, RVtone.1, U1.2 (-), U1.6 (-), U1.9 (-)
- new net VCC: C9.2, Q1.3 (C), R3.2, R4.2, R7.2, U1.11 (V-)
- new net VSS: C10.2, U1.4 (V+)
Other:
- note added: "out"
- note added: "trig in"

Commit message: VCO draft
Additions:
- Draft of VCO module
Changes:
- None
Removals:
- None
Parts:
- removed C10: 100n, symbol Device:C
- removed D4: LED, symbol Device:LED
- removed RV1: 10K, symbol Device:R_Potentiometer
- removed RVdecay: 500K (panel: Decay), symbol Device:R_Potentiometer
- removed RVlevel: 10K (panel: Level), symbol Device:R_Potentiometer
- removed RVpitch: 100K (panel: Pitch), symbol Device:R_Potentiometer
- removed RVtone: 5K (panel: Tone), symbol Device:R_Potentiometer
- added C11: 100n, Capacitor_THT:C_Disc_D5.0mm_W2.5mm_P5.00mm, symbol Device:C
- added C8: 15n, Capacitor_THT:C_Disc_D5.0mm_W2.5mm_P5.00mm, symbol Device:C
- added Q3, Q4, Q5: 2N3904, Package_TO_SOT_THT:TO-92_Inline, symbol Transistor_BJT:2N3904
- added R21: 10K, Resistor_THT:R_Axial_DIN0207_L6.3mm_D2.5mm_P10.16mm_Horizontal, symbol Device:R
- added R22: 100K, Resistor_THT:R_Axial_DIN0207_L6.3mm_D2.5mm_P10.16mm_Horizontal, symbol Device:R
- added R23: 4.7K, Resistor_THT:R_Axial_DIN0207_L6.3mm_D2.5mm_P10.16mm_Horizontal, symbol Device:R
- added RV2: 100K, Potentiometer_THT:Potentiometer_Alps_RK09K_Single_Vertical, symbol Device:R_Potentiometer
- added RV3: 5K, Potentiometer_THT:Potentiometer_Alps_RK09K_Single_Vertical, symbol Device:R_Potentiometer
- added RV4: 500K, Potentiometer_THT:Potentiometer_Alps_RK09K_Single_Vertical, symbol Device:R_Potentiometer
- added RV5: 10K, Potentiometer_THT:Potentiometer_Alps_RK09K_Single_Vertical, symbol Device:R_Potentiometer
- C1, C2, C3, C4, C5, C7, C9: footprint (none) -> Capacitor_THT:C_Disc_D5.0mm_W2.5mm_P5.00mm
- C6: footprint (none) -> Capacitor_THT:CP_Radial_D5.0mm_P2.00mm
- D1, D2, D3: footprint (none) -> Diode_THT:D_DO-35_SOD27_P7.62mm_Horizontal
- J3: renamed from R1; value 22K -> POWER; footprint (none) -> Connector_PinHeader_2.54mm:PinHeader_1x03_P2.54mm_Vertical; symbol Device:R -> Connector_Generic:Conn_01x03
- Q1, Q2: footprint (none) -> Package_TO_SOT_THT:TO-92_Inline
- R10, R11, R12, R13, R14, R15, R16, R17, R18, R19, R2, R4, R5, R6, R7, R8, R9: footprint (none) -> Resistor_THT:R_Axial_DIN0207_L6.3mm_D2.5mm_P10.16mm_Horizontal
- R20: value 1K -> 100K; footprint (none) -> Resistor_THT:R_Axial_DIN0207_L6.3mm_D2.5mm_P10.16mm_Horizontal
- R3: value 47K -> 4.7K; footprint (none) -> Resistor_THT:R_Axial_DIN0207_L6.3mm_D2.5mm_P10.16mm_Horizontal
- U1: footprint (none) -> Package_DIP:DIP-14_W7.62mm
Connections:
- net GND: now also C2.2, J3.2 (Pin_2), Q2.1 (E), R2.2, R20.2, R5.2, U1.10 (+), U1.12 (+), U1.5 (+), C11.2, Q3.1 (E), Q4.1 (E), Q5.1 (E), R23.2, RV2.3, RV5.3; no longer C9.1, D3.1 (K), Q2.3 (C), R2.1, U1.2 (-), U1.6 (-), U1.9 (-)
- net VCC: now also C9.1, J3.1 (Pin_1), Q1.1 (E), R3.1, R4.1, R7.1, U1.4 (V+); no longer C9.2, Q1.3 (C), R3.2, R4.2, R7.2, U1.11 (V-)
- net VSS: now also C9.2, J3.3 (Pin_3), U1.11 (V-); no longer U1.4 (V+)
- net at R20.1: now also C1.1, D1.1 (K)
- net at Q2.2 (B): now also R5.1, R6.2; no longer U1.13 (-)
- net at R15.1: now also R13.2, R14.2, U1.6 (-), RV4.1, RV4.2
- net at C3.2: now also D2.2 (A), R8.1; no longer R7.1
- net at R13.1: now also C5.2, R12.2, R14.1, U1.1, RV3.1; no longer R14.2
- net at C4.1: now also R12.1, U1.2 (-); no longer C5.2
- net at C7.1: now also C11.1, RV3.2, RV3.3; no longer R16.2
- net at R9.1: now also C3.1, R7.2, Q4.3 (C)
- net at R19.1: now also R17.2, U1.8
- new net: C6.2, R11.2, R15.2, U1.7
- new net: C2.1, Q2.3 (C), Q4.2 (B), R4.2
- new net: C4.2, C5.1, R10.2, R11.1, R8.2
- new net: C8.1, Q1.3 (C), R22.1, R6.1
- new net: C8.2, R22.2, R23.1, U1.3 (+)
- new net: D1.2 (A), J3.1 (Pin_1)
- new net: J3.2 (Pin_2), Q3.2 (B), R2.1
- new net: R18.1, RV5.2
- new net: R17.1, R18.2, U1.9 (-)
- new net: C6.1, RV4.3
- new net: C7.2, D3.2 (A), RV5.1
- new net: Q5.3 (C), R10.1, RV2.1, RV2.2
- new net: D3.1 (K), R16.1
- new net: Q1.2 (B), R21.1, R3.2
- new net: J3.1 (Pin_1), R16.2
- new net: C1.2, J3.1 (Pin_1)
- new net: U1.13 (-), U1.14
- new net: Q3.3 (C), R21.2
- new net: Q5.2 (B), R9.2
- new net: J3.1 (Pin_1), R19.2
Other:
- note added: "808 KICK"
- note added: "J1 trigger, J2 output, J3 power (VCC / GND / VSS)."
- note added: "Layout follows KiCAD/references/808kick/808kick-reference-eddybergman.JPG"
- note added: "M4TM version (Juanito Moore circuit), after the Eddy Bergman reference drawing"
- note added: "Panel pots: RV2 Pitch 100K; RV3 Tone 5K; RV4 Decay 500K; RV5 Level 10K."
- note added: "SW1: header for off-board SPST clipper switch."
- note added: "clipper"
- note added: "decay"
- note added: "level"
- note added: "pitch"
- note added: "supply"
- note added: "tone"
- note added: "trig"
- note added: "unused op amp"
- note removed: "trig in"
- title: (none) -> 808 Kick - M4TM / Eddy Bergman reference
- moved on the sheet: C1, C2, C3, C4, C5, C6, C7, C9, D1, D2, D3, Q1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
