File: KiCAD/current-modules/synth-allmodules/VCO.kicad_sch (KiCad schematic)
At the start: 0 parts

Commit message: VCO draft
Additions:
- Draft of VCO module
Changes:
- None
Removals:
- None
Parts:
- added C201: 100p, Capacitor_THT:C_Disc_D5.0mm_W2.5mm_P5.00mm, symbol Device:C
- added C202: 470p, Capacitor_THT:C_Disc_D5.0mm_W2.5mm_P5.00mm, symbol Device:C
- added C203, C204, C205, C206, C207, C208, C209: 10n, Capacitor_THT:C_Disc_D5.0mm_W2.5mm_P5.00mm, symbol Device:C
- added C210: 100n, Capacitor_THT:C_Disc_D5.0mm_W2.5mm_P5.00mm, symbol Device:C
- added C211: 220n, Capacitor_THT:C_Disc_D5.0mm_W2.5mm_P5.00mm, symbol Device:C
- added C212, C213: 10u, Capacitor_THT:CP_Radial_D5.0mm_P2.00mm, symbol Device:C_Polarized
- added D201, D202, D203: 1N4148, Diode_THT:D_DO-35_SOD27_P7.62mm_Horizontal, symbol Diode:1N4148
- added J201: 1V/OCT, Connector_PinHeader_2.54mm:PinHeader_1x02_P2.54mm_Vertical, symbol Connector_Generic:Conn_01x02
- added J202: EXP FM, Connector_PinHeader_2.54mm:PinHeader_1x02_P2.54mm_Vertical, symbol Connector_Generic:Conn_01x02
- added J203: LIN FM, Connector_PinHeader_2.54mm:PinHeader_1x02_P2.54mm_Vertical, symbol Connector_Generic:Conn_01x02
- added J204: HARD SYNC, Connector_PinHeader_2.54mm:PinHeader_1x02_P2.54mm_Vertical, symbol Connector_Generic:Conn_01x02
- added J205: TRIANGLE, Connector_PinHeader_2.54mm:PinHeader_1x02_P2.54mm_Vertical, symbol Connector_Generic:Conn_01x02
- added J206: RAMPOID, Connector_PinHeader_2.54mm:PinHeader_1x02_P2.54mm_Vertical, symbol Connector_Generic:Conn_01x02
- added J207: SAW, Connector_PinHeader_2.54mm:PinHeader_1x02_P2.54mm_Vertical, symbol Connector_Generic:Conn_01x02
- added J208: PWM, Connector_PinHeader_2.54mm:PinHeader_1x02_P2.54mm_Vertical, symbol Connector_Generic:Conn_01x02
- added J209: SINE, Connector_PinHeader_2.54mm:PinHeader_1x02_P2.54mm_Vertical, symbol Connector_Generic:Conn_01x02
- added J210: PULSE, Connector_PinHeader_2.54mm:PinHeader_1x02_P2.54mm_Vertical, symbol Connector_Generic:Conn_01x02
- added J211: +12 / GND / -12, Connector_PinHeader_2.54mm:PinHeader_1x03_P2.54mm_Vertical, symbol Connector_Generic:Conn_01x03
- added Q201, Q202, Q203, Q204, Q205: 2N3904, Package_TO_SOT_THT:TO-92_Inline, symbol Transistor_BJT:2N3904
- added R202, R203: 390R, Resistor_THT:R_Axial_DIN0207_L6.3mm_D2.5mm_P10.16mm_Horizontal, symbol Device:R
- added R204, R205, R206, R207: 1k, Resistor_THT:R_Axial_DIN0207_L6.3mm_D2.5mm_P10.16mm_Horizontal, symbol Device:R
- added R208, R210, R211, R212, R213: 2.2k, Resistor_THT:R_Axial_DIN0207_L6.3mm_D2.5mm_P10.16mm_Horizontal, symbol Device:R
- added R209: 2k, Resistor_THT:R_Axial_DIN0207_L6.3mm_D2.5mm_P10.16mm_Horizontal, symbol Device:R
- added R214: 4.7k, Resistor_THT:R_Axial_DIN0207_L6.3mm_D2.5mm_P10.16mm_Horizontal, symbol Device:R
- added R215, R216, R217: 10k, Resistor_THT:R_Axial_DIN0207_L6.3mm_D2.5mm_P10.16mm_Horizontal, symbol Device:R
- added R218, R219: 15k, Resistor_THT:R_Axial_DIN0207_L6.3mm_D2.5mm_P10.16mm_Horizontal, symbol Device:R
- added R220: 12k, Resistor_THT:R_Axial_DIN0207_L6.3mm_D2.5mm_P10.16mm_Horizontal, symbol Device:R
- added R221: 18k, Resistor_THT:R_Axial_DIN0207_L6.3mm_D2.5mm_P10.16mm_Horizontal, symbol Device:R
- added R222: 33k, Resistor_THT:R_Axial_DIN0207_L6.3mm_D2.5mm_P10.16mm_Horizontal, symbol Device:R
- added R224, R225, R226: 75k, Resistor_THT:R_Axial_DIN0207_L6.3mm_D2.5mm_P10.16mm_Horizontal, symbol Device:R
- added R227, R228, R229, R230, R231, R232, R233, R234, R235: 100k, Resistor_THT:R_Axial_DIN0207_L6.3mm_D2.5mm_P10.16mm_Horizontal, symbol Device:R
- added R248, R249: 120k, Resistor_THT:R_Axial_DIN0207_L6.3mm_D2.5mm_P10.16mm_Horizontal, symbol Device:R
- added R250, R251, R252: 220k, Resistor_THT:R_Axial_DIN0207_L6.3mm_D2.5mm_P10.16mm_Horizontal, symbol Device:R
- added R254: 1.5M, Resistor_THT:R_Axial_DIN0207_L6.3mm_D2.5mm_P10.16mm_Horizontal, symbol Device:R
- added R255: 2.2M, Resistor_THT:R_Axial_DIN0207_L6.3mm_D2.5mm_P10.16mm_Horizontal, symbol Device:R
- added R256: 3.3M, Resistor_THT:R_Axial_DIN0207_L6.3mm_D2.5mm_P10.16mm_Horizontal, symbol Device:R
- added RV201: 100R, Potentiometer_THT:Potentiometer_Bourns_3296W_Vertical, symbol Device:R_Potentiometer
- added RV223: 50k, Potentiometer_THT:Potentiometer_Bourns_3296W_Vertical, symbol Device:R_Potentiometer
- added RV236, RV237, RV238, RV239, RV240, RV241: 100k, Potentiometer_THT:Potentiometer_Bourns_3296W_Vertical, symbol Device:R_Potentiometer
- added RV242, RV243, RV244, RV245, RV246, RV247: 100k, Potentiometer_THT:Potentiometer_Alps_RK09K_Single_Vertical, symbol Device:R_Potentiometer
- added RV253: 500k, Potentiometer_THT:Potentiometer_Alps_RK09K_Single_Vertical, symbol Device:R_Potentiometer
- added S201: AC/DC, Connector_PinHeader_2.54mm:PinHeader_1x02_P2.54mm_Vertical, symbol Switch:SW_SPST
- added U201: CD4046B, Package_DIP:DIP-16_W7.62mm, symbol 4xxx:4046
- added U202: LF442, VCO_EasyEDA:PDIP-8_L9.3-W6.4-P2.54-LS7.9-BL-1, symbol VCO_EasyEDA:LF442ACN_NOPB
- added U203, U204: TL074, Package_DIP:DIP-14_W7.62mm, symbol Amplifier_Operational:TL074
Connections:
- new net: Q205.2 (B), R211.1
- new net: R225.1, RV237.1, U203.1, U203.2 (-)
- new net: C203.2, U201.7 (C2), U203.3 (+)
- new net: R235.2, R249.1, R252.2, U204.13 (-)
- new net: R249.2, U204.14, U204.9 (-)
- new net: J210.1 (Pin_1), R208.1, R213.2
- new net: R228.1, RV242.2
- new net: R209.1, R227.2, R228.2, R229.2, R256.2, U202.2 (IN1-)
- new net: C203.1, U201.6 (C1), U203.5 (+)
- new net: R212.2, R255.1, U204.10 (+)
- new net: R213.1, R255.2, U204.8
- new net: D202.1 (K), R215.1
- new net: R215.2, RV236.1
- new net: C202.1, J204.1 (Pin_1)
- new net: Q205.1 (E), R203.2, RV223.3
- new net: Q205.3 (C), R217.2, R219.1, U204.5 (+)
- new net: R207.1, R212.1, R218.2, U204.7
- new net: J209.1 (Pin_1), R207.2
- new net: D201.1 (K), D202.2 (A)
- new net: R224.1, R226.1, U203.6 (-), U203.7
- new net: R224.2, R233.2, R248.1, U203.10 (+)
- new net: R251.1, RV240.2
- new net: R225.2, R226.2, R234.1, R251.2, U203.13 (-)
- new net: C201.2, R220.1, RV236.2, RV236.3, U202.7 (OUT2)
- new net: Q201.1 (E), Q202.1 (E), R220.2
- new net: R209.2, RV201.1, U202.1 (OUT1)
- new net: D201.2 (A), Q201.2 (B), RV201.2
- new net: R202.1, RV201.3
- new net: Q204.3 (C), R216.2, R218.1, U204.6 (-)
- new net: R256.1, RV244.2
- new net: C202.2, R231.1
- new net: D203.1 (K), Q203.2 (B), R231.2
- new net: J205.1 (Pin_1), R204.2
- new net: J201.1 (Pin_1), R227.1
- new net: J206.1 (Pin_1), R205.2
- new net: R252.1, RV247.2
- new net: R230.1, RV245.2
- new net: C201.1, Q201.3 (C), R230.2, R254.2, U202.6 (IN2-)
- new net: R222.1, RV237.2
- new net: Q204.1 (E), R203.1, RV223.1
- new net: Q204.2 (B), R210.1, RV241.2, RV241.3
- new net: R250.1, RV238.2
- new net: R222.2, R232.1, R250.2, U203.9 (-)
- new net: R206.1, R234.2, RV253.3, U203.14
- new net: J202.1 (Pin_1), RV242.1
- new net: Q203.3 (C), R214.2, U201.3 (RefIn)
- new net: R204.1, R232.2, RV241.1, RV253.1, U203.8
- new net: R229.1, RV243.2
- new net: J207.1 (Pin_1), R206.2
- new net: C211.1, J203.1 (Pin_1), S201.1 (A)
- new net: C211.2, RV245.1, S201.2 (B)
- new net: RV239.1, U201.4 (FOUT)
- new net: R233.1, RV239.2
- new net: R221.1, RV223.2
- new net: RV253.2, U204.3 (+)
- new net: J208.1 (Pin_1), RV246.1
- new net: R205.1, U204.1, U204.2 (-)
- new net: Q202.3 (C), U201.11 (R1)
- new net: U201.2 (PC1), U201.5 (Inh)
- new net: R235.1, RV246.2
- new net +12V: C204.1, C206.1, C208.1, C210.1, C212.1, J211.1 (Pin_1), R214.1, R216.1, R217.1, R254.1, RV238.1, RV243.1, RV244.1, RV247.1, U201.14 (SigIn), U201.16 (VDD), U201.9 (VCOin), U202.8 (V+), U203.4 (V+), U204.4 (V+)
- new net -12V: C205.2, C207.2, C209.2, C213.2, J211.3 (Pin_3), R221.2, RV240.1, RV243.3, RV244.3, RV247.3, U202.4 (V-), U203.11 (V-), U204.11 (V-)
- new net GND: C204.2, C205.1, C206.2, C207.1, C208.2, C209.1, C210.2, C212.2, C213.1, D203.2 (A), J201.2 (Pin_2), J202.2 (Pin_2), J203.2 (Pin_2), J204.2 (Pin_2), J205.2 (Pin_2), J206.2 (Pin_2), J207.2 (Pin_2), J208.2 (Pin_2), J209.2 (Pin_2), J210.2 (Pin_2), J211.2 (Pin_2), Q202.2 (B), Q203.1 (E), R202.2, R208.2, R210.2, R211.2, R219.2, R248.2, RV237.3, RV238.3, RV239.3, RV240.3, RV242.3, RV245.3, RV246.3, U201.8 (VSS), U202.3 (IN1+), U202.5 (IN2+), U203.12 (+), U204.12 (+)
- no-connect marks 0 -> 5
Other:
- note added: "AC/DC"
- note added: "C204-C209 10n and C212/C213 10u: close to U202-U204 supply pins. C210 100n at U201."
- note added: "COARSE"
- note added: "Calibration: RV201 V/oct; RV236 HF; RV237/239 triangle connect; RV238 triangle offset; RV240 saw offset; RV241 round; RV223 symmetry."
- note added: "EXP FM ATTEN"
- note added: "FINE"
- note added: "HF TRIM"
- note added: "INITIAL WIDTH"
- note added: "J201-J210: two-pin headers to panel jacks (pin 1 signal, pin 2 ground). S201: off-board AC/DC switch."
- note added: "LIN FM ATTEN"
- note added: "Layout follows KiCAD/references/VCO/VCO-reference-thomashenry.jpg"
- note added: "PWM ATTEN"
- note added: "R209: 2k, +3500 ppm/C tempco."
- note added: "SAW OFFSET"
- note added: "SINE ROUND"
- note added: "SINE SYMMETRY"
- note added: "SKEW"
- note added: "Source refs Rn / Cn / Qn / Jn map to 200+n; IC1-IC4 map to U201-U204; pots use RV."
- note added: "TRIANGLE CONNECT 1"
- note added: "TRIANGLE CONNECT 2"
- note added: "TRIANGLE OFFSET"
- note added: "Thermally couple Q201 / Q202 and R209."
- note added: "Thomas Henry, last rev June 13, 2010 (12 V version)"
- note added: "V/OCT TRIM"
- note added: "X-4046 VCO"
- title: (none) -> X-4046 VCO - Thomas Henry
