File: KiCAD/current-modules/synth-allmodules/ADSR.kicad_sch (KiCad schematic)
At the start: 42 parts, among them Q1 BC547, Q2 BC547, Q3 BC547, Q4 BC547, SW1 SW_Push, U1 ICM7555xP, U2 TL074

Commit message: ADSR finished
Additions:
- Remaining component values for ADSR
Changes:
- None
Removals:
- None
Parts:
- C67, C68: value C_Polarized -> 100u
- R13, R14: value R -> 100K
- R15, R16: value R -> 1K
- R17: value R -> 33K
- R18: value R -> 4.7K
- RV5: value R_Potentiometer -> 100K lin
Changed lines of the file:
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@@
 			)
 		)
-		(property "Value" "R"
+		(property "Value" "1K"
 			(at 222.25 72.39 90)
 			(show_name no)
@@
 			)
 		)
-		(property "Value" "R"
+		(property "Value" "100K"
 			(at 180.34 100.3299 0)
 			(show_name no)
@@
 			)
 		)
-		(property "Value" "R"
+		(property "Value" "100K"
 			(at 200.66 72.39 90)
 			(show_name no)
@@
 			)
 		)
-		(property "Value" "R_Potentiometer"
+		(property "Value" "100K lin"
 			(at 224.79 102.8699 0)
 			(show_name no)
@@
 			)
 		)
-		(property "Value" "R"
+		(property "Value" "4.7K"
 			(at 256.54 140.9699 0)
 			(show_name no)
@@
 			)
 		)
-		(property "Value" "R"
+		(property "Value" "33K"
 			(at 205.74 137.1599 0)
 			(show_name no)
@@
 			)
 		)
-		(property "Value" "C_Polarized"
+		(property "Value" "100u"
 			(at 238.76 53.7209 0)
 			(show_name no)
@@
 			)
 		)
-		(property "Value" "R"
+		(property "Value" "1K"
 			(at 222.25 123.19 90)
 			(show_name no)
@@
 			)
 		)
-		(property "Value" "C_Polarized"
+		(property "Value" "100u"
 			(at 238.76 42.2909 0)
 			(show_name no)

Commit message: First Draft of 808
Additions:
- Draft of 808 Kick module
Changes:
- None
Removals:
- None
Parts:
- C2: value C_Polarized -> 1u
Changed lines of the file:
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@@
 			)
 		)
-		(property "Value" "C_Polarized"
+		(property "Value" "1u"
 			(at 168.91 164.2109 0)
 			(show_name no)

Commit message: Audio Jacks
Additions:
- Audio jack IOs for all sheets
Changes:
- None
Removals:
- None
Parts:
- added J4: GATE_IN, Connector_PinHeader_2.54mm:PinHeader_1x02_P2.54mm_Vertical, symbol Connector_Generic:Conn_01x02
- added J5: OUTPUT, Connector_PinHeader_2.54mm:PinHeader_1x02_P2.54mm_Vertical, symbol Connector_Generic:Conn_01x02
- added J6: ATTEN_OUT, Connector_PinHeader_2.54mm:PinHeader_1x02_P2.54mm_Vertical, symbol Connector_Generic:Conn_01x02
Connections:
- net GND: now also J4.2 (Pin_2), J5.2 (Pin_2), J6.2 (Pin_2)
- net at R3.1: now also J4.1 (Pin_1)
- net at R15.1: now also J6.1 (Pin_1)
- net at R16.1: now also J5.1 (Pin_1)
Other:
- note added: "attenuverter out"
