File: KiCAD/current-modules/synth-allmodules/LFO.kicad_sch (KiCad schematic)
At the start: 57 parts, among them Q10 BC547, Q11 BC547, U12 TL074, U13 TL074, U14 TL072

Commit message: Audio Jacks
Additions:
- Audio jack IOs for all sheets
Changes:
- None
Removals:
- None
Parts:
- added J20: PULSE_1, Connector_PinHeader_2.54mm:PinHeader_1x02_P2.54mm_Vertical, symbol Connector_Generic:Conn_01x02
- added J21: TRI_SAW_1, Connector_PinHeader_2.54mm:PinHeader_1x02_P2.54mm_Vertical, symbol Connector_Generic:Conn_01x02
- added J22: SQUARE_1, Connector_PinHeader_2.54mm:PinHeader_1x02_P2.54mm_Vertical, symbol Connector_Generic:Conn_01x02
- added J23: VAR_1, Connector_PinHeader_2.54mm:PinHeader_1x02_P2.54mm_Vertical, symbol Connector_Generic:Conn_01x02
- added J24: PULSE_2, Connector_PinHeader_2.54mm:PinHeader_1x02_P2.54mm_Vertical, symbol Connector_Generic:Conn_01x02
- added J25: TRI_SAW_2, Connector_PinHeader_2.54mm:PinHeader_1x02_P2.54mm_Vertical, symbol Connector_Generic:Conn_01x02
- added J26: SQUARE_2, Connector_PinHeader_2.54mm:PinHeader_1x02_P2.54mm_Vertical, symbol Connector_Generic:Conn_01x02
- added J27: VAR_2, Connector_PinHeader_2.54mm:PinHeader_1x02_P2.54mm_Vertical, symbol Connector_Generic:Conn_01x02
Connections:
- net GND: now also J20.2 (Pin_2), J21.2 (Pin_2), J22.2 (Pin_2), J23.2 (Pin_2), J24.2 (Pin_2), J25.2 (Pin_2), J26.2 (Pin_2), J27.2 (Pin_2)
- net at R79.1, R80.2: now also J22.1 (Pin_1)
- net at R84.2, R97.1: now also J24.1 (Pin_1)
- net at R93.1, R94.2: now also J26.1 (Pin_1)
- net at R88.1, R89.2: now also J25.1 (Pin_1)
- net at R70.1, R71.2: now also J20.1 (Pin_1)
- net at R96.1: now also J27.1 (Pin_1)
- net at R74.1, R75.2: now also J21.1 (Pin_1)
- net at R82.1: now also J23.1 (Pin_1)
