File: KiCAD/current-modules/synth-allmodules/VCA.kicad_sch (KiCad schematic)
At the start: 45 parts, among them Q9 2N3906, SW15 SW_SPST, SW16 SW_SPST, SW5 SW_SPST, U10 TL071, U11 CA3080, U9 TL072

Commit message: Audio Jacks
Additions:
- Audio jack IOs for all sheets
Changes:
- None
Removals:
- None
Parts:
- added J13: AUDIO_1, Connector_PinHeader_2.54mm:PinHeader_1x02_P2.54mm_Vertical, symbol Connector_Generic:Conn_01x02
- added J14: AUDIO_2, Connector_PinHeader_2.54mm:PinHeader_1x02_P2.54mm_Vertical, symbol Connector_Generic:Conn_01x02
- added J15: AUDIO_3, Connector_PinHeader_2.54mm:PinHeader_1x02_P2.54mm_Vertical, symbol Connector_Generic:Conn_01x02
- added J16: ENVELOPE, Connector_PinHeader_2.54mm:PinHeader_1x02_P2.54mm_Vertical, symbol Connector_Generic:Conn_01x02
- added J17: VAR_CV, Connector_PinHeader_2.54mm:PinHeader_1x02_P2.54mm_Vertical, symbol Connector_Generic:Conn_01x02
- added J18: MAX_OUT, Connector_PinHeader_2.54mm:PinHeader_1x02_P2.54mm_Vertical, symbol Connector_Generic:Conn_01x02
- added J19: LINE_OUT, Connector_PinHeader_2.54mm:PinHeader_1x02_P2.54mm_Vertical, symbol Connector_Generic:Conn_01x02
Connections:
- net GND: now also J13.2 (Pin_2), J14.2 (Pin_2), J15.2 (Pin_2), J16.2 (Pin_2), J17.2 (Pin_2), J18.2 (Pin_2), J19.2 (Pin_2)
- net at C29.1, SW15.1 (A): now also J14.1 (Pin_1)
- net at C26.1, SW5.1 (A): now also J13.1 (Pin_1)
- net at R61.2: now also J18.1 (Pin_1)
- net at RV30.1: now also J17.1 (Pin_1)
- net at C30.1, SW16.1 (A): now also J15.1 (Pin_1)
- net at R66.1: now also J16.1 (Pin_1)
- net at C32.2: now also J19.1 (Pin_1)
Other:
- note removed: "Variable CV"
